File: pcb/flowcontrol-v0.1/flowcontrol-v0.1.sch (KiCad schematic (older format))
At the start: 9 parts

Commit message: update PCB
Parts:
- added C1, C2, C3: 22pF, symbol Device:C
- added J6: Molex 4 Pin, symbol Connector:Conn_01x04_Female
- added J7: 4 Pin DRGB LED, symbol Connector:Conn_01x04_Male
- added R3, R4: 10k Ω, symbol Device:R
- added Y1: 12Mhz Crystal, symbol Device:Crystal
- J3, J4: renamed from J?; value Temp Sensor -> Temp Sensor (10k Thermistor)
- gave numbers to parts that had none: 7
Connections:
- net labels added: D+, D-, DIN, GP0, GP1, GP10, GP11, GPO
- net labels removed: +12V, +5V
- wire segments 0 -> 19
Other:
- moved on the sheet: J1, J2, J3, J4, J5, R1, R2, U2

Commit message: start new revision of PCB with integrated CH340G
Parts:
- removed C1, C2, C3: 22pF, symbol Device:C
- removed J5: Internal USB, symbol Connector:Conn_01x04_Male
- removed U2: CH340G, symbol ch34x:CH340G
- removed Y1: 12Mhz Crystal, symbol Device:Crystal
- added C? (x3): 100n?, 0603_N, symbol CH340G_D-SUN-V3.0-rescue:C
- added C?: 10u?, 0603_N, symbol CH340G_D-SUN-V3.0-rescue:C
- added C? (x2): 22p?, 0603_N, symbol CH340G_D-SUN-V3.0-rescue:C
- added CON?: USB, symbol CH340G_D-SUN-V3.0-rescue:connUsb
- added D? (x2): LL4148, SMA_N, symbol CH340G_D-SUN-V3.0-rescue:diode
- added D? (x3): LED, SMA_N, symbol CH340G_D-SUN-V3.0-rescue:diode_LED
- added Q?: 12MHz, symbol CH340G_D-SUN-V3.0-rescue:XT_2pin
- added R? (x4): 1k5, 0603_N, symbol CH340G_D-SUN-V3.0-rescue:R
- added U?: CH340G, SOIC-16_N, symbol CH340G_D-SUN-V3.0-rescue:CH340G
- J1, J2, J7: symbol Connector:Conn_01x04_Male -> flowcontrol-v0.1-rescue:Conn_01x04_Male-Connector
- J3, J4: symbol Connector:Conn_01x02_Female -> flowcontrol-v0.1-rescue:Conn_01x02_Female-Connector
- J6: symbol Connector:Conn_01x04_Female -> flowcontrol-v0.1-rescue:Conn_01x04_Female-Connector
- R1, R2: symbol Device:R_Small -> flowcontrol-v0.1-rescue:R_Small-Device
- R3, R4: symbol Device:R -> flowcontrol-v0.1-rescue:R-Device
- U1: symbol Pico_rp2040:PICO_RP2040 -> flowcontrol-v0.1-rescue:PICO_RP2040-Pico_rp2040
Connections:
- net 12v: no longer J6.4 (Pin_4)
- net 5v: no longer J6.1 (Pin_1), U1.39 (VSYS)
- net GND: now also C?.2, C?.2, C?.2, C?.2, C?.2, C?.2, CON?.0 (GND), CON?.4 (GND), R?.2, U?.1 (GND)
- net GP0: now also R?.2
- net GP1: now also D?.1 (A), U?.3 (RxD)
- net 3.3v renamed +3V3
- net +3V3: now also C?.1, C?.1, D?.1 (A), D?.2 (C), R?.1, R?.1, U?.16 (VCC), U?.4 (3V)
- new net: CON?.3 (D+), U?.5 (D+)
- new net: CON?.2 (D-), U?.6 (D-)
- new net: C?.1, Q?.1, U?.7 (XI)
- new net: C?.1, Q?.3, U?.8 (XO)
- new net: D?.1 (A), D?.2 (C)
- new net: D?.1 (A), R?.1
- new net: D?.2 (C), R?.2 (x2)
- new net +5V: C?.1, C?.1, CON?.1 (5V), D?.2 (C), J6.1 (Pin_1), U1.39 (VSYS)
- new net TxD: D?.1 (A), R?.1, U?.2 (TxD)
- no-connect marks 0 -> 7
Other:
- moved on the sheet: J1, J2, J3, J4, J6, J7, R1, R2, R3, R4, U1
