File: pcb/src/flowcontrol-v0.1.kicad_pcb (KiCad board)
At the start: 2 copper layers, 89 x 59 mm, 34 parts, among them J1 Fan 1, J2 Fan 2, J3 Temp Sensor (10k Thermistor), J4 Temp Sensor (10k Thermistor), J5 Internal USB, J6 Molex 4 Pin, J7 4 Pin DRGB LED, SW1 K2-1102SP-C4SC-04, U1 PICO_RP2040, U2 CH340G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

Commit message: add revision 3 PCB (#47)
* add revision 3 PCB

* remove test firmwares
Parts:
- moved J6 15.6 mm to (174.4, 73.1), turned to 180 degrees
Connections:
- D4 pad 1: GP1 -> GP0
- J5 pad 1: (no net) -> Net-(J5-Pad1)
- J5 pad 10: (no net) -> Net-(J5-Pad10)
- J5 pad 2: (no net) -> +5V
- J5 pad 3: (no net) -> Net-(J5-Pad3)
- J5 pad 5: (no net) -> Net-(J5-Pad5)
- J5 pad 7: (no net) -> Net-(J5-Pad7)
- J5 pad 9: (no net) -> Net-(J5-Pad9)
- J6 pad 1: +5V -> +12V
- J6 pad 4: +12V -> +5V
- R5 pad 2: GP0 -> GP1
- U2 pad 3: GP1 -> GP0
Routing:
- net GND: track 209.1 -> 223.3 mm
- net +5V: track 189.3 -> 181.3 mm
- net GP0: track 69.0 -> 65.2 mm, vias 0 -> 3
- net GP1: track 64.0 -> 67.3 mm, vias 3 -> 0
Other:
- board text added: "reset"
- board text added: "rev 0.3"
- board text removed: "rev 0.2"
