File: pcb/src/flowcontrol.kicad_pcb (KiCad board)
At the start: 2 copper layers, 89 x 59 mm, 34 parts, among them J1 Fan 1, J2 Fan 2, J3 Temp Sensor (10k Thermistor), J4 Temp Sensor (10k Thermistor), J5 Internal USB, J6 Molex 4 Pin, J7 4 Pin DRGB LED, SW1 K2-1102SP-C4SC-04, U1 PICO_RP2040, U2 CH340G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

Commit message: create revision 4 PCB
Parts:
- moved R4 94.4 mm to (259.8, 77.5)
- moved J4 94.4 mm to (247.1, 96.5)
- moved R1 94.4 mm to (248.4, 77.5)
- moved J3 94.4 mm to (258.5, 96.5)
- moved R2 94.4 mm to (252.2, 77.5)
- moved R3 94.4 mm to (256.0, 77.5)
- moved SW1 94.4 mm to (256.1, 85.1)
- moved J7 90.7 mm to (245.9, 63.7)
- moved J2 73.8 mm to (228.1, 50.0)
- moved J1 73.8 mm to (228.1, 31.0)
- moved J5 72.1 mm to (50.4, 24.9)
- moved C1 67.7 mm to (47.7, 76.1)
- moved C2 67.7 mm to (50.3, 76.1)
- moved C3 67.7 mm to (52.8, 76.1)
- moved C4 67.7 mm to (55.4, 76.1)
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Routing:
- net GND: track 223.3 -> 0.00 mm, vias 8 -> 0
- net +5V: track 181.3 -> 0.00 mm
- net GP11: track 102.5 -> 0.00 mm
- net GP10: track 94.2 -> 0.00 mm
- net GP26: track 76.8 -> 0.00 mm, vias 2 -> 0
- net GP7: track 74.1 -> 0.00 mm, vias 2 -> 0
- net GP1: track 67.3 -> 0.00 mm
- net GP6: track 65.5 -> 0.00 mm, vias 2 -> 0
- net GP0: track 65.2 -> 0.00 mm, vias 3 -> 0
- net +3V3: track 63.8 -> 0.00 mm, vias 10 -> 0
- net GP27: track 54.6 -> 0.00 mm, vias 2 -> 0
- net Net-(C4-Pad1): track 53.4 -> 0.00 mm, vias 2 -> 0
- net Net-(D3-Pad2): track 53.0 -> 0.00 mm
- net Net-(C5-Pad1): track 51.2 -> 0.00 mm, vias 2 -> 0
- net TxD: track 50.9 -> 0.00 mm
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
Commit message: add gerbers
Parts:
- added J10: Fan 1, Connector_PinHeader_2.54mm:PinHeader_1x04_P2.54mm_Horizontal, F.Cu at (111.5, 74.9)
- added J11: Fan 2, Connector_PinHeader_2.54mm:PinHeader_1x04_P2.54mm_Horizontal, F.Cu at (126.0, 74.9)
- added J8: Fan 5, Connector_PinHeader_2.54mm:PinHeader_1x04_P2.54mm_Horizontal, F.Cu at (133.6, 112.8)
- added J9: Fan 6, Connector_PinHeader_2.54mm:PinHeader_1x04_P2.54mm_Horizontal, F.Cu at (147.8, 112.8)
- added R10: 10k Ω, Resistor_SMD:R_0603_1608Metric, F.Cu at (165.0, 86.4)
- added R11: 10k Ω, Resistor_SMD:R_0603_1608Metric, F.Cu at (165.0, 84.1)
- added R12: 10k Ω, Resistor_SMD:R_0603_1608Metric, F.Cu at (169.9, 84.1)
- added R9: 10k Ω, Resistor_SMD:R_0603_1608Metric, F.Cu at (169.9, 86.4)
- J1: value Fan 1 -> Fan 3
- J2: value Fan 2 -> Fan 4
- J3, J4: footprint Connector_JST:JST_XH_B2B-XH-A_1x02_P2.50mm_Vertical -> Connector_JST:JST_XH_S2B-XH-A-1_1x02_P2.50mm_Horizontal
- J5: footprint Connector_PinSocket_2.54mm:PinSocket_2x05_P2.54mm_Vertical -> Connector_PinSocket_2.54mm:PinSocket_2x05_P2.54mm_Horizontal
- J6: footprint Connector_TE-Connectivity:TE_MATE-N-LOK_350211-1_1x04_P5.08mm_Vertical -> LibraryLoader:641737-1
- J7: footprint Connector_PinHeader_2.54mm:PinHeader_1x04_P2.54mm_Vertical -> Connector_PinHeader_2.54mm:PinHeader_1x04_P2.54mm_Horizontal
- moved J5 135.3 mm to (155.2, 110.5)
- moved D2 132.5 mm to (165.8, 106.7)
- moved D1 128.2 mm to (158.0, 106.7)
- moved J2 125.3 mm to (119.6, 112.8), turned to 270 degrees
- moved R6 120.2 mm to (169.9, 95.4)
- moved C1 119.6 mm to (165.2, 98.5), turned to 0 degrees
- moved R5 119.2 mm to (165.0, 95.4)
- moved C2 117.6 mm to (165.2, 101.1), turned to 0 degrees
- moved C4 116.6 mm to (169.8, 98.5), turned to 0 degrees
- moved C3 115.7 mm to (165.2, 103.6), turned to 0 degrees
- moved C5 114.7 mm to (169.8, 101.1), turned to 0 degrees
- moved C6 112.8 mm to (169.8, 103.6), turned to 0 degrees
- moved Y1 112.5 mm to (157.2, 80.0), turned to 180 degrees
- moved R8 112.3 mm to (169.9, 93.2)
- moved R7 111.3 mm to (165.0, 93.2)
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Connections:
- net RUN renamed Net-(SW1-Pad1)
- J1 pad 2: GP10 -> GP23
- J2 pad 2: GP11 -> GP24
- R3 pad 1: +5V -> +3V3
- R3 pad 2: GP10 -> GP23
- R4 pad 1: +5V -> +3V3
- R4 pad 2: GP11 -> GP24
- U1 pad 11: Net-(U1-Pad11) -> GP8
- U1 pad 12: Net-(U1-Pad12) -> GP9
- U1 pad 14: GP10 -> Net-(U1-Pad14)
- U1 pad 15: GP11 -> Net-(U1-Pad15)
- U1 pad 21: Net-(U1-Pad21) -> GP26
- U1 pad 22: Net-(U1-Pad22) -> GP25
- U1 pad 24: Net-(U1-Pad24) -> GP24
- U1 pad 25: Net-(U1-Pad25) -> GP23
- U1 pad 26: Net-(U1-Pad26) -> GP22
- U1 pad 27: Net-(U1-Pad27) -> GP21
- U1 pad 6: Net-(U1-Pad6) -> GP4
- U1 pad 7: Net-(U1-Pad7) -> GP5
Routing:
- net +5V: track 0.00 -> 239.4 mm, vias 0 -> 2
- net +12V: track 0.00 -> 227.8 mm
- net TxD: track 0.00 -> 147.5 mm, vias 0 -> 2
- net GP26: track 0.00 -> 134.1 mm, vias 0 -> 5
- net Net-(D3-Pad2): track 0.00 -> 112.1 mm, vias 0 -> 2
- net Net-(D5-Pad1): track 0.00 -> 97.0 mm, vias 0 -> 2
- net GP0: track 0.00 -> 95.7 mm, vias 0 -> 2
- net GP5: track 0.00 -> 93.0 mm
- net GP6: track 0.00 -> 90.7 mm
- net Net-(D4-Pad2): track 0.00 -> 90.1 mm, vias 0 -> 2
- net GP4: track 0.00 -> 87.8 mm
- net GP21: track 0.00 -> 83.2 mm, vias 0 -> 3
- net GP24: track 0.00 -> 73.3 mm, vias 0 -> 3
- net GND: track 0.00 -> 73.0 mm, vias 0 -> 2
- net DIN: track 0.00 -> 72.6 mm
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Other:
- board text added: "FAN1"
- board text added: "FAN2"
- board text added: "FAN3"
- board text added: "FAN4"
- board text added: "FAN5"
- board text added: "FAN6"
- board text added: "INTERNAL USB"
- board text added: "POWER"
- board text added: "RX"
- board text added: "SENSOR1"
- board text added: "SENSOR2"
- board text added: "TX"
- board text added: "revision 4"
- board text removed: "USB"
- board text removed: "fan 1"
- board text removed: "fan 2"
- board text removed: "rev 0.3"
- board text removed: "temp sensor 1"
- board text removed: "temp sensor 2"
