File: pcb/src/flowcontrol.sch (KiCad schematic (older format))
At the start: 30 parts, among them J1 Fan 1, J2 Fan 2, J3 Temp Sensor (10k Thermistor), J4 Temp Sensor (10k Thermistor), J5 Internal USB, J6 Molex 4 Pin, J7 4 Pin DRGB LED, SW1 K2-1102SP-C4SC-04, U1 PICO_RP2040, U2 CH340G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

Commit message: create revision 4 PCB
Parts:
- added J10: Fan 1, Connector_PinHeader_2.54mm:PinHeader_1x04_P2.54mm_Horizontal, symbol flowcontrol-rescue:Conn_01x04_Male-Connector
- added J11: Fan 2, Connector_PinHeader_2.54mm:PinHeader_1x04_P2.54mm_Horizontal, symbol flowcontrol-rescue:Conn_01x04_Male-Connector
- added J8: Fan 5, Connector_PinHeader_2.54mm:PinHeader_1x04_P2.54mm_Horizontal, symbol flowcontrol-rescue:Conn_01x04_Male-Connector
- added J9: Fan 6, Connector_PinHeader_2.54mm:PinHeader_1x04_P2.54mm_Horizontal, symbol flowcontrol-rescue:Conn_01x04_Male-Connector
- added R10, R11, R12, R9: 10k Ω, Resistor_SMD:R_0603_1608Metric, symbol flowcontrol-rescue:R-Device
- C1, C2, C3, C4, C5, C6: symbol flowcontrol-v0.1-rescue:C-CH340G_D-SUN-V3.0-rescue -> flowcontrol-rescue:C-CH340G_D-SUN-V3.0-rescue
- D1, D2: symbol flowcontrol-v0.1-rescue:diode-CH340G_D-SUN-V3.0-rescue -> flowcontrol-rescue:diode-CH340G_D-SUN-V3.0-rescue
- D3, D4, D5: symbol flowcontrol-v0.1-rescue:diode_LED-CH340G_D-SUN-V3.0-rescue -> flowcontrol-rescue:diode_LED-CH340G_D-SUN-V3.0-rescue
- J1: value Fan 1 -> Fan 3; symbol flowcontrol-v0.1-rescue:Conn_01x04_Male-Connector -> flowcontrol-rescue:Conn_01x04_Male-Connector
- J2: value Fan 2 -> Fan 4; symbol flowcontrol-v0.1-rescue:Conn_01x04_Male-Connector -> flowcontrol-rescue:Conn_01x04_Male-Connector
- J3, J4: footprint Connector_JST:JST_XH_B2B-XH-A_1x02_P2.50mm_Vertical -> Connector_JST:JST_XH_S2B-XH-A-1_1x02_P2.50mm_Horizontal; symbol flowcontrol-v0.1-rescue:Conn_01x02_Female-Connector -> flowcontrol-rescue:Conn_01x02_Female-Connector
- J5: footprint Connector_PinSocket_2.54mm:PinSocket_2x05_P2.54mm_Vertical -> Connector_PinSocket_2.54mm:PinSocket_2x05_P2.54mm_Horizontal
- J6: footprint Connector_TE-Connectivity:TE_MATE-N-LOK_350211-1_1x04_P5.08mm_Vertical -> LibraryLoader:641737-1; symbol flowcontrol-v0.1-rescue:Conn_01x04_Female-Connector -> SamacSys_Parts:641737-1
- J7: footprint Connector_PinHeader_2.54mm:PinHeader_1x04_P2.54mm_Vertical -> Connector_PinHeader_2.54mm:PinHeader_1x04_P2.54mm_Horizontal; symbol flowcontrol-v0.1-rescue:Conn_01x04_Male-Connector -> flowcontrol-rescue:Conn_01x04_Male-Connector
- R1, R2: symbol flowcontrol-v0.1-rescue:R_Small-Device -> flowcontrol-rescue:R_Small-Device
- R3, R4: symbol flowcontrol-v0.1-rescue:R-Device -> flowcontrol-rescue:R-Device
- R5, R6, R7, R8: symbol flowcontrol-v0.1-rescue:R-CH340G_D-SUN-V3.0-rescue -> flowcontrol-rescue:R-CH340G_D-SUN-V3.0-rescue
- U1: symbol flowcontrol-v0.1-rescue:PICO_RP2040-Pico_rp2040 -> flowcontrol-rescue:PICO_RP2040-Pico_rp2040
- U2: symbol flowcontrol-v0.1-rescue:CH340G-CH340G_D-SUN-V3.0-rescue -> flowcontrol-rescue:CH340G-CH340G_D-SUN-V3.0-rescue
Connections:
- net labels added: GP21, GP22, GP23, GP24, GP25, GP4, GP5, GP8, GP9
- net labels removed: GP10, GP11, RUN
- wire segments 78 -> 94
Other:
- moved on the sheet: J1, J2, J7, R3, R4, SW1, U1

Commit message: add gerbers
Parts:
- C1, C2, C3, C4, C5, C6: symbol flowcontrol-rescue:C-CH340G_D-SUN-V3.0-rescue -> flowcontrol-rescue:C-CH340G_D-SUN-V3.0-rescue-flowcontrol-rescue
- D1, D2: symbol flowcontrol-rescue:diode-CH340G_D-SUN-V3.0-rescue -> flowcontrol-rescue:diode-CH340G_D-SUN-V3.0-rescue-flowcontrol-rescue
- D3, D4, D5: symbol flowcontrol-rescue:diode_LED-CH340G_D-SUN-V3.0-rescue -> flowcontrol-rescue:diode_LED-CH340G_D-SUN-V3.0-rescue-flowcontrol-rescue
- J1, J10, J11, J2, J7, J8, J9: symbol flowcontrol-rescue:Conn_01x04_Male-Connector -> flowcontrol-rescue:Conn_01x04_Male-Connector-flowcontrol-rescue
- J3, J4: symbol flowcontrol-rescue:Conn_01x02_Female-Connector -> flowcontrol-rescue:Conn_01x02_Female-Connector-flowcontrol-rescue
- R1, R2: symbol flowcontrol-rescue:R_Small-Device -> flowcontrol-rescue:R_Small-Device-flowcontrol-rescue
- R10, R11, R12, R3, R4, R9: symbol flowcontrol-rescue:R-Device -> flowcontrol-rescue:R-Device-flowcontrol-rescue
- R5, R6, R7, R8: symbol flowcontrol-rescue:R-CH340G_D-SUN-V3.0-rescue -> flowcontrol-rescue:R-CH340G_D-SUN-V3.0-rescue-flowcontrol-rescue
- U1: symbol flowcontrol-rescue:PICO_RP2040-Pico_rp2040 -> flowcontrol-rescue:PICO_RP2040-Pico_rp2040-flowcontrol-rescue
- U2: symbol flowcontrol-rescue:CH340G-CH340G_D-SUN-V3.0-rescue -> flowcontrol-rescue:CH340G-CH340G_D-SUN-V3.0-rescue-flowcontrol-rescue
